File: MozzaCircuit/MozzaCircuit.kicad_sch (KiCad schematic)
At the start: 17 parts, among them J1 8P8C_both_sides, U1 MCP23017_ML, U2 MCP23017_ML

Commit message: init pcb
Parts:
- JPB2, JPB3, JPB4, JPB6, JPB7, JPB8, JPF2, JPF3, JPF4, JPF6, JPF7, JPF8: footprint (none) -> Jumper:SolderJumper-2_P1.3mm_Open_TrianglePad1.0x1.5mm
Changed lines of the file:
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@@
       (effects (font (size 1.27 1.27)) hide)
     )
-    (property "Footprint" "" (id 2) (at 59.69 66.04 0)
+    (property "Footprint" "Jumper:SolderJumper-2_P1.3mm_Open_TrianglePad1.0x1.5mm" (id 2) (at 59.69 66.04 0)
       (effects (font (size 1.27 1.27)) hide)
     )
@@
       (effects (font (size 1.27 1.27)) hide)
     )
-    (property "Footprint" "" (id 2) (at 59.69 86.36 0)
+    (property "Footprint" "Jumper:SolderJumper-2_P1.3mm_Open_TrianglePad1.0x1.5mm" (id 2) (at 59.69 86.36 0)
       (effects (font (size 1.27 1.27)) hide)
     )
@@
       (effects (font (size 1.27 1.27)) hide)
     )
-    (property "Footprint" "" (id 2) (at 59.69 83.82 0)
+    (property "Footprint" "Jumper:SolderJumper-2_P1.3mm_Open_TrianglePad1.0x1.5mm" (id 2) (at 59.69 83.82 0)
       (effects (font (size 1.27 1.27)) hide)
     )
@@
       (effects (font (size 1.27 1.27)) hide)
     )
-    (property "Footprint" "" (id 2) (at 59.69 91.44 0)
+    (property "Footprint" "Jumper:SolderJumper-2_P1.3mm_Open_TrianglePad1.0x1.5mm" (id 2) (at 59.69 91.44 0)
       (effects (font (size 1.27 1.27)) hide)
     )
@@
       (effects (font (size 1.27 1.27)) hide)
     )
-    (property "Footprint" "" (id 2) (at 59.69 60.96 0)
+    (property "Footprint" "Jumper:SolderJumper-2_P1.3mm_Open_TrianglePad1.0x1.5mm" (id 2) (at 59.69 60.96 0)
       (effects (font (size 1.27 1.27)) hide)
     )
@@
       (effects (font (size 1.27 1.27)) hide)
     )
-    (property "Footprint" "" (id 2) (at 59.69 73.66 0)
+    (property "Footprint" "Jumper:SolderJumper-2_P1.3mm_Open_TrianglePad1.0x1.5mm" (id 2) (at 59.69 73.66 0)
       (effects (font (size 1.27 1.27)) hide)
     )
@@
       (effects (font (size 1.27 1.27)) hide)
     )
-    (property "Footprint" "" (id 2) (at 59.69 71.12 0)
+    (property "Footprint" "Jumper:SolderJumper-2_P1.3mm_Open_TrianglePad1.0x1.5mm" (id 2) (at 59.69 71.12 0)
       (effects (font (size 1.27 1.27)) hide)
     )
@@
       (effects (font (size 1.27 1.27)) hide)
     )
-    (property "Footprint" "" (id 2) (at 59.69 63.5 0)
+    (property "Footprint" "Jumper:SolderJumper-2_P1.3mm_Open_TrianglePad1.0x1.5mm" (id 2) (at 59.69 63.5 0)
       (effects (font (size 1.27 1.27)) hide)
     )
@@
       (effects (font (size 1.27 1.27)) hide)
     )
-    (property "Footprint" "" (id 2) (at 59.69 68.58 0)
+    (property "Footprint" "Jumper:SolderJumper-2_P1.3mm_Open_TrianglePad1.0x1.5mm" (id 2) (at 59.69 68.58 0)
       (effects (font (size 1.27 1.27)) hide)
     )
@@
       (effects (font (size 1.27 1.27)) hide)
     )
-    (property "Footprint" "" (id 2) (at 59.69 78.74 0)
+    (property "Footprint" "Jumper:SolderJumper-2_P1.3mm_Open_TrianglePad1.0x1.5mm" (id 2) (at 59.69 78.74 0)
       (effects (font (size 1.27 1.27)) hide)
     )
@@
       (effects (font (size 1.27 1.27)) hide)
     )
-    (property "Footprint" "" (id 2) (at 59.69 88.9 0)
+    (property "Footprint" "Jumper:SolderJumper-2_P1.3mm_Open_TrianglePad1.0x1.5mm" (id 2) (at 59.69 88.9 0)
       (effects (font (size 1.27 1.27)) hide)
     )
@@
       (effects (font (size 1.27 1.27)) hide)
     )
-    (property "Footprint" "" (id 2) (at 59.69 81.28 0)
+    (property "Footprint" "Jumper:SolderJumper-2_P1.3mm_Open_TrianglePad1.0x1.5mm" (id 2) (at 59.69 81.28 0)
       (effects (font (size 1.27 1.27)) hide)
     )
@@
     )
     (path "/91cb7703-e23f-4a57-bc86-173230b77ba5"
-      (reference "JPB2") (unit 1) (value "SolderJumper_2_Open") (footprint "")
+      (reference "JPB2") (unit 1) (value "SolderJumper_2_Open") (footprint "Jumper:SolderJumper-2_P1.3mm_Open_TrianglePad1.0x1.5mm")
     )
     (path "/b9696c75-eb80-4fce-a706-cc2c622d7bbc"
-      (reference "JPB3") (unit 1) (value "SolderJumper_2_Open") (footprint "")
+      (reference "JPB3") (unit 1) (value "SolderJumper_2_Open") (footprint "Jumper:SolderJumper-2_P1.3mm_Open_TrianglePad1.0x1.5mm")
     )
     (path "/68562b54-861e-4aad-a091-c03666ae4751"
-      (reference "JPB4") (unit 1) (value "SolderJumper_2_Open") (footprint "")
+      (reference "JPB4") (unit 1) (value "SolderJumper_2_Open") (footprint "Jumper:SolderJumper-2_P1.3mm_Open_TrianglePad1.0x1.5mm")
     )
     (path "/f6ff7905-fa8c-464b-91b7-4a5893c9649d"
-      (reference "JPB6") (unit 1) (value "SolderJumper_2_Open") (footprint "")
+      (reference "JPB6") (unit 1) (value "SolderJumper_2_Open") (footprint "Jumper:SolderJumper-2_P1.3mm_Open_TrianglePad1.0x1.5mm")
     )
     (path "/1d15cbb9-d2f5-4857-83ba-68568b253bb6"
-      (reference "JPB7") (unit 1) (value "SolderJumper_2_Open") (footprint "")
+      (reference "JPB7") (unit 1) (value "SolderJumper_2_Open") (footprint "Jumper:SolderJumper-2_P1.3mm_Open_TrianglePad1.0x1.5mm")
     )
     (path "/57309842-c78d-4f8d-9a1d-d3070a1a62c9"
-      (reference "JPB8") (unit 1) (value "SolderJumper_2_Open") (footprint "")
+      (reference "JPB8") (unit 1) (value "SolderJumper_2_Open") (footprint "Jumper:SolderJumper-2_P1.3mm_Open_TrianglePad1.0x1.5mm")
     )
     (path "/d976194f-3238-4d59-a9dc-1448b4cb2d56"
-      (reference "JPF2") (unit 1) (value "SolderJumper_2_Open") (footprint "")
+      (reference "JPF2") (unit 1) (value "SolderJumper_2_Open") (footprint "Jumper:SolderJumper-2_P1.3mm_Open_TrianglePad1.0x1.5mm")
     )
     (path "/4320a7b8-49d1-4e5f-b1c3-489ef77493a1"
-      (reference "JPF3") (unit 1) (value "SolderJumper_2_Open") (footprint "")
+      (reference "JPF3") (unit 1) (value "SolderJumper_2_Open") (footprint "Jumper:SolderJumper-2_P1.3mm_Open_TrianglePad1.0x1.5mm")
     )
     (path "/cea82208-4ffc-4096-a15b-39178b693c3c"
-      (reference "JPF4") (unit 1) (value "SolderJumper_2_Open") (footprint "")
+      (reference "JPF4") (unit 1) (value "SolderJumper_2_Open") (footprint "Jumper:SolderJumper-2_P1.3mm_Open_TrianglePad1.0x1.5mm")
     )
     (path "/73639fda-9dd4-424c-b8aa-23771b935260"
-      (reference "JPF6") (unit 1) (value "SolderJumper_2_Open") (footprint "")
+      (reference "JPF6") (unit 1) (value "SolderJumper_2_Open") (footprint "Jumper:SolderJumper-2_P1.3mm_Open_TrianglePad1.0x1.5mm")
     )
     (path "/1105f6a9-9c52-471f-84c8-a06aa02d172c"
-      (reference "JPF7") (unit 1) (value "SolderJumper_2_Open") (footprint "")
+      (reference "JPF7") (unit 1) (value "SolderJumper_2_Open") (footprint "Jumper:SolderJumper-2_P1.3mm_Open_TrianglePad1.0x1.5mm")
     )
     (path "/62b9a5da-77cb-4614-bc4f-3c34d8c2c649"
-      (reference "JPF8") (unit 1) (value "SolderJumper_2_Open") (footprint "")
+      (reference "JPF8") (unit 1) (value "SolderJumper_2_Open") (footprint "Jumper:SolderJumper-2_P1.3mm_Open_TrianglePad1.0x1.5mm")
     )
     (path "/096fe43d-bb63-4e85-b408-1b08ff8375d2/898502e1-7835-4255-8cf5-ffc25ec8ae82"

Commit message: started place and route
Parts:
- removed U2: MCP23017_ML, 00_KeyParts:QFN-28-1EP_6x6mm_P0.65mm_EP4.25x4.25mm_Hand_NoTP, symbol Interface_Expansion:MCP23017_ML
- added U2: MCP23017_ML_NoTP, 00_KeyParts:QFN-28-1EP_6x6mm_P0.65mm_EP4.25x4.25mm_Hand_NoTP, symbol 00_KeyParts:MCP23017_ML_NoTP
Connections:
- net 3V3: now also U2.11 (A0), U2.5 (VDD)
- net COL1: now also U2.17 (GPA0)
- net COL2: now also U2.18 (GPA1)
- net COL3: now also U2.19 (GPA2)
- net COL4: now also U2.20 (GPA3)
- net COL5: now also U2.21 (GPA4)
- net COL6: now also U2.22 (GPA5)
- net COL7: now also U2.23 (GPA6)
- net COL8: now also U2.24 (GPA7)
- net GND: now also U2.12 (A1), U2.13 (A2), U2.6 (VSS)
- net NRST: now also U2.14 (~{RESET})
- net REA: now also U2.2 (GPB5)
- net REB: now also U2.3 (GPB6)
- net ROW1: now also U2.25 (GPB0)
- net ROW2: now also U2.26 (GPB1)
- net ROW3: now also U2.27 (GPB2)
- net ROW4: now also U2.28 (GPB3)
- net ROW5: now also U2.1 (GPB4)
- net SCK: now also U2.8 (SCK)
- net SDA: now also U2.9 (SDA)
Changed lines of the file:
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@@
   (junction (at 55.88 63.5) (diameter 0) (color 0 0 0 0)
-  )
-  (junction (at 114.3 165.1) (diameter 0) (color 0 0 0 0)
   )
   (junction (at 55.88 68.58) (diameter 0) (color 0 0 0 0)
@@
     (stroke (width 0) (type default) (color 0 0 0 0))
   )
-  (wire (pts (xy 111.76 165.1) (xy 114.3 165.1))
-    (stroke (width 0) (type default) (color 0 0 0 0))
-  )
   (wire (pts (xy 55.88 88.9) (xy 55.88 91.44))
     (stroke (width 0) (type default) (color 0 0 0 0))
@@
     (pin "1")
   )
+  (symbol (lib_id "00_KeyParts:MCP23017_ML_NoTP") (at 114.3 137.16 0) (unit 1)
+    (in_bom yes) (on_board yes) (fields_autoplaced)
+    (property "Reference" "U2" (id 0) (at 116.3194 109.22 0)
+      (effects (font (size 1.27 1.27)) (justify left))
+    )
+    (property "Value" "MCP23017_ML_NoTP" (id 1) (at 116.3194 111.76 0)
+      (effects (font (size 1.27 1.27)) (justify left))
+    )
+    (property "Footprint" "00_KeyParts:QFN-28-1EP_6x6mm_P0.65mm_EP4.25x4.25mm_Hand_NoTP" (id 2) (at 119.38 162.56 0)
+      (effects (font (size 1.27 1.27)) (justify left) hide)
+    )
+    (property "Datasheet" "http://ww1.microchip.com/downloads/en/DeviceDoc/20001952C.pdf" (id 3) (at 119.38 165.1 0)
+      (effects (font (size 1.27 1.27)) (justify left) hide)
+    )
+    (pin "1")
+    (pin "10")
+    (pin "11")
+    (pin "12")
+    (pin "13")
+    (pin "14")
+    (pin "15")
+    (pin "16")
+    (pin "17")
+    (pin "18")
+    (pin "19")
+    (pin "2")
+    (pin "20")
+    (pin "21")
+    (pin "22")
+    (pin "23")
+    (pin "24")
+    (pin "25")
+    (pin "26")
+    (pin "27")
+    (pin "28")
+    (pin "3")
+    (pin "4")
+    (pin "5")
+    (pin "6")
+    (pin "7")
+    (pin "8")
+    (pin "9")
+  )
   (symbol (lib_id "power:PWR_FLAG") (at 38.1 33.02 90) (unit 1)
     (in_bom yes) (on_board yes) (fields_autoplaced)
@@
     (pin "1")
   )
-  (symbol (lib_id "Interface_Expansion:MCP23017_ML") (at 114.3 137.16 0) (unit 1)
+  (symbol (lib_id "Interface_Expansion:MCP23017_ML") (at 50.8 137.16 0) (unit 1)
     (in_bom yes) (on_board yes) (fields_autoplaced)
-    (property "Reference" "U2" (id 0) (at 116.3194 109.22 0)
+    (property "Reference" "U1" (id 0) (at 52.8194 109.22 0)
       (effects (font (size 1.27 1.27)) (justify left))
     )
-    (property "Value" "MCP23017_ML" (id 1) (at 116.3194 111.76 0)
+    (property "Value" "MCP23017_ML" (id 1) (at 52.8194 111.76 0)
       (effects (font (size 1.27 1.27)) (justify left))
     )
-    (property "Footprint" "00_KeyParts:QFN-28-1EP_6x6mm_P0.65mm_EP4.25x4.25mm_Hand_NoTP" (id 2) (at 119.38 162.56 0)
-      (effects (font (size 1.27 1.27)) (justify left) hide)
-    )
-    (property "Datasheet" "http://ww1.microchip.com/downloads/en/DeviceDoc/20001952C.pdf" (id 3) (at 119.38 165.1 0)
+    (property "Footprint" "00_KeyParts:QFN-28-1EP_6x6mm_P0.65mm_EP4.25x4.25mm_Hand" (id 2) (at 55.88 162.56 0)
+      (effects (font (size 1.27 1.27)) (justify left) hide)
+    )
+    (property "Datasheet" "http://ww1.microchip.com/downloads/en/DeviceDoc/20001952C.pdf" (id 3) (at 55.88 165.1 0)
       (effects (font (size 1.27 1.27)) (justify left) hide)
     )
@@
     (pin "9")
   )
-  (symbol (lib_id "Interface_Expansion:MCP23017_ML") (at 50.8 137.16 0) (unit 1)
-    (in_bom yes) (on_board yes) (fields_autoplaced)
-    (property "Reference" "U1" (id 0) (at 52.8194 109.22 0)
-      (effects (font (size 1.27 1.27)) (justify left))
-    )
-    (property "Value" "MCP23017_ML" (id 1) (at 52.8194 111.76 0)
-      (effects (font (size 1.27 1.27)) (justify left))
-    )
-    (property "Footprint" "00_KeyParts:QFN-28-1EP_6x6mm_P0.65mm_EP4.25x4.25mm_Hand" (id 2) (at 55.88 162.56 0)
-      (effects (font (size 1.27 1.27)) (justify left) hide)
-    )
-    (property "Datasheet" "http://ww1.microchip.com/downloads/en/DeviceDoc/20001952C.pdf" (id 3) (at 55.88 165.1 0)
-      (effects (font (size 1.27 1.27)) (justify left) hide)
-    )
-    (pin "1")
-    (pin "10")
-    (pin "11")
-    (pin "12")
-    (pin "13")
-    (pin "14")
-    (pin "15")
-    (pin "16")
-    (pin "17")
-    (pin "18")
-    (pin "19")
-    (pin "2")
-    (pin "20")
-    (pin "21")
-    (pin "22")
-    (pin "23")
-    (pin "24")
-    (pin "25")
-    (pin "26")
-    (pin "27")
-    (pin "28")
-    (pin "29")
-    (pin "3")
-    (pin "4")
-    (pin "5")
-    (pin "6")
-    (pin "7")
-    (pin "8")
-    (pin "9")
-  )
   (symbol (lib_id "power:GND") (at 96.52 154.94 270) (unit 1)
     (in_bom yes) (on_board yes)
@@
       (reference "#FLG0104") (unit 1) (value "PWR_FLAG") (footprint "")
     )
+    (path "/096fe43d-bb63-4e85-b408-1b08ff8375d2/f2bf7d47-8676-46a0-86b8-34a144e7baf8"
+      (reference "#FLG0105") (unit 1) (value "PWR_FLAG") (footprint "")
+    )
     (path "/33e8908d-03d7-4408-82f3-027acfa8898f"
       (reference "#PWR0101") (unit 1) (value "GND") (footprint "")
@@
       (reference "C2") (unit 1) (value "C_Small") (footprint "00_KeyParts:C_2012")
     )
-    (path "/096fe43d-bb63-4e85-b408-1b08ff8375d2/a4afcd60-a18d-4cba-b572-9557deda77cf"
-      (reference "C11") (unit 1) (value "0.1u") (footprint "00_KeyParts:C_2012_rev")
-    )
     (path "/096fe43d-bb63-4e85-b408-1b08ff8375d2/3f07d010-f525-4889-b35d-2c573f2fe087"
       (reference "C12") (unit 1) (value "C_Small") (footprint "00_KeyParts:C_2012_rev")
@@
       (reference "C13") (unit 1) (value "C_Small") (footprint "00_KeyParts:C_2012_rev")
     )
-    (path "/096fe43d-bb63-4e85-b408-1b08ff8375d2/a62c955f-8568-4568-a3c5-9a877d4c73d7"
-      (reference "C14") (unit 1) (value "C_Small") (footprint "00_KeyParts:C_2012_rev")
-    )
     (path "/096fe43d-bb63-4e85-b408-1b08ff8375d2/4ae6a39a-2fb7-4f23-8b07-007f392c0bef"
       (reference "C15") (unit 1) (value "C_Small") (footprint "00_KeyParts:C_2012_rev")
     )
     (path "/096fe43d-bb63-4e85-b408-1b08ff8375d2/822dbaaa-2882-483b-af09-fc71a09ac544"
-      (reference "C21") (unit 1) (value "C_Small") (footprint "00_KeyParts:C_2012_rev")
+      (reference "C21") (unit 1) (value "0.1u") (footprint "00_KeyParts:C_2012_rev")
     )
     (path "/096fe43d-bb63-4e85-b408-1b08ff8375d2/3f3609fc-d8af-4236-a520-81f6014410d1"
@@
       (reference "D84") (unit 1) (value "D_Small") (footprint "00_KeyParts:D_SOD-323_both_sides")
     )
+    (path "/096fe43d-bb63-4e85-b408-1b08ff8375d2/c15344b4-ae2e-4b67-bee4-ff0e49a0c8b6"
+      (reference "DL1") (unit 1) (value "D_Small") (footprint "00_KeyParts:D_SOD-323_both_sides")
+    )
     (path "/afde2c83-3cd9-4387-a068-f4bd55db6222"
       (reference "J1") (unit 1) (value "8P8C_both_sides") (footprint "00_KeyParts:RJ45_Molex_0955032884_both_sides")
@@
       (reference "U1") (unit 1) (value "MCP23017_ML") (footprint "00_KeyParts:QFN-28-1EP_6x6mm_P0.65mm_EP4.25x4.25mm_Hand")
     )
-    (path "/21c35884-09fe-4da8-a010-f2b680d013b0"
-      (reference "U2") (unit 1) (value "MCP23017_ML") (footprint "00_KeyParts:QFN-28-1EP_6x6mm_P0.65mm_EP4.25x4.25mm_Hand_NoTP")
-    )
-  )
+    (path "/1e0176b1-6fe6-436c-b636-4b5d1babcb7c"
+      (reference "U2") (unit 1) (value "MCP23017_ML_NoTP") (footprint "00_KeyParts:QFN-28-1EP_6x6mm_P0.65mm_EP4.25x4.25mm_Hand_NoTP")
+    )
+  )
