File: MozzaCircuit/MozzaCircuit.kicad_sch (KiCad schematic)
At the start: 16 parts, among them J1 8P8C_both_sides, U1 MCP23017_ML, U2 MCP23017_ML_NoTP

Commit message: edgecuts, gnd vias, screw holes
Parts:
- added H1, H2, H3, H4, H5, H6, H7, H8: MountingHole, 00_KeyParts:SpacerHole_M2_4mm, symbol Mechanical:MountingHole
Changed lines of the file:
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@@
     (pin "9")
   )
+  (symbol (lib_id "Mechanical:MountingHole") (at 139.7 69.85 0) (unit 1)
+    (in_bom yes) (on_board yes) (fields_autoplaced)
+    (property "Reference" "H2" (id 0) (at 142.24 68.5799 0)
+      (effects (font (size 1.27 1.27)) (justify left))
+    )
+    (property "Value" "MountingHole" (id 1) (at 142.24 71.1199 0)
+      (effects (font (size 1.27 1.27)) (justify left))
+    )
+    (property "Footprint" "00_KeyParts:SpacerHole_M2_4mm" (id 2) (at 139.7 69.85 0)
+      (effects (font (size 1.27 1.27)) hide)
+    )
+    (property "Datasheet" "~" (id 3) (at 139.7 69.85 0)
+      (effects (font (size 1.27 1.27)) hide)
+    )
+  )
   (symbol (lib_id "power:GND") (at 96.52 154.94 270) (unit 1)
     (in_bom yes) (on_board yes)
@@
     )
     (pin "1")
+  )
+  (symbol (lib_id "Mechanical:MountingHole") (at 158.75 76.2 0) (unit 1)
+    (in_bom yes) (on_board yes) (fields_autoplaced)
+    (property "Reference" "H7" (id 0) (at 161.29 74.9299 0)
+      (effects (font (size 1.27 1.27)) (justify left))
+    )
+    (property "Value" "MountingHole" (id 1) (at 161.29 77.4699 0)
+      (effects (font (size 1.27 1.27)) (justify left))
+    )
+    (property "Footprint" "00_KeyParts:SpacerHole_M2_4mm" (id 2) (at 158.75 76.2 0)
+      (effects (font (size 1.27 1.27)) hide)
+    )
+    (property "Datasheet" "~" (id 3) (at 158.75 76.2 0)
+      (effects (font (size 1.27 1.27)) hide)
+    )
   )
   (symbol (lib_id "Device:C_Small") (at 171.45 116.84 0) (unit 1)
@@
     (pin "1")
   )
+  (symbol (lib_id "Mechanical:MountingHole") (at 139.7 76.2 0) (unit 1)
+    (in_bom yes) (on_board yes) (fields_autoplaced)
+    (property "Reference" "H3" (id 0) (at 142.24 74.9299 0)
+      (effects (font (size 1.27 1.27)) (justify left))
+    )
+    (property "Value" "MountingHole" (id 1) (at 142.24 77.4699 0)
+      (effects (font (size 1.27 1.27)) (justify left))
+    )
+    (property "Footprint" "00_KeyParts:SpacerHole_M2_4mm" (id 2) (at 139.7 76.2 0)
+      (effects (font (size 1.27 1.27)) hide)
+    )
+    (property "Datasheet" "~" (id 3) (at 139.7 76.2 0)
+      (effects (font (size 1.27 1.27)) hide)
+    )
+  )
+  (symbol (lib_id "Mechanical:MountingHole") (at 158.75 69.85 0) (unit 1)
+    (in_bom yes) (on_board yes) (fields_autoplaced)
+    (property "Reference" "H6" (id 0) (at 161.29 68.5799 0)
+      (effects (font (size 1.27 1.27)) (justify left))
+    )
+    (property "Value" "MountingHole" (id 1) (at 161.29 71.1199 0)
+      (effects (font (size 1.27 1.27)) (justify left))
+    )
+    (property "Footprint" "00_KeyParts:SpacerHole_M2_4mm" (id 2) (at 158.75 69.85 0)
+      (effects (font (size 1.27 1.27)) hide)
+    )
+    (property "Datasheet" "~" (id 3) (at 158.75 69.85 0)
+      (effects (font (size 1.27 1.27)) hide)
+    )
+  )
   (symbol (lib_id "power:GND") (at 88.9 66.04 90) (unit 1)
     (in_bom yes) (on_board yes) (fields_autoplaced)
@@
     (pin "2")
   )
+  (symbol (lib_id "Mechanical:MountingHole") (at 158.75 63.5 0) (unit 1)
+    (in_bom yes) (on_board yes) (fields_autoplaced)
+    (property "Reference" "H5" (id 0) (at 161.29 62.2299 0)
+      (effects (font (size 1.27 1.27)) (justify left))
+    )
+    (property "Value" "MountingHole" (id 1) (at 161.29 64.7699 0)
+      (effects (font (size 1.27 1.27)) (justify left))
+    )
+    (property "Footprint" "00_KeyParts:SpacerHole_M2_4mm" (id 2) (at 158.75 63.5 0)
+      (effects (font (size 1.27 1.27)) hide)
+    )
+    (property "Datasheet" "~" (id 3) (at 158.75 63.5 0)
+      (effects (font (size 1.27 1.27)) hide)
+    )
+  )
+  (symbol (lib_id "Mechanical:MountingHole") (at 158.75 82.55 0) (unit 1)
+    (in_bom yes) (on_board yes) (fields_autoplaced)
+    (property "Reference" "H8" (id 0) (at 161.29 81.2799 0)
+      (effects (font (size 1.27 1.27)) (justify left))
+    )
+    (property "Value" "MountingHole" (id 1) (at 161.29 83.8199 0)
+      (effects (font (size 1.27 1.27)) (justify left))
+    )
+    (property "Footprint" "00_KeyParts:SpacerHole_M2_4mm" (id 2) (at 158.75 82.55 0)
+      (effects (font (size 1.27 1.27)) hide)
+    )
+    (property "Datasheet" "~" (id 3) (at 158.75 82.55 0)
+      (effects (font (size 1.27 1.27)) hide)
+    )
+  )
   (symbol (lib_id "power:PWR_FLAG") (at 38.1 29.21 90) (unit 1)
     (in_bom yes) (on_board yes) (fields_autoplaced)
@@
     )
     (pin "1")
+  )
+  (symbol (lib_id "Mechanical:MountingHole") (at 139.7 63.5 0) (unit 1)
+    (in_bom yes) (on_board yes) (fields_autoplaced)
+    (property "Reference" "H1" (id 0) (at 142.24 62.2299 0)
+      (effects (font (size 1.27 1.27)) (justify left))
+    )
+    (property "Value" "MountingHole" (id 1) (at 142.24 64.7699 0)
+      (effects (font (size 1.27 1.27)) (justify left))
+    )
+    (property "Footprint" "00_KeyParts:SpacerHole_M2_4mm" (id 2) (at 139.7 63.5 0)
+      (effects (font (size 1.27 1.27)) hide)
+    )
+    (property "Datasheet" "~" (id 3) (at 139.7 63.5 0)
+      (effects (font (size 1.27 1.27)) hide)
+    )
   )
   (symbol (lib_id "power:GND") (at 38.1 36.83 90) (unit 1)
@@
     (pin "2")
   )
+  (symbol (lib_id "Mechanical:MountingHole") (at 139.7 82.55 0) (unit 1)
+    (in_bom yes) (on_board yes) (fields_autoplaced)
+    (property "Reference" "H4" (id 0) (at 142.24 81.2799 0)
+      (effects (font (size 1.27 1.27)) (justify left))
+    )
+    (property "Value" "MountingHole" (id 1) (at 142.24 83.8199 0)
+      (effects (font (size 1.27 1.27)) (justify left))
+    )
+    (property "Footprint" "00_KeyParts:SpacerHole_M2_4mm" (id 2) (at 139.7 82.55 0)
+      (effects (font (size 1.27 1.27)) hide)
+    )
+    (property "Datasheet" "~" (id 3) (at 139.7 82.55 0)
+      (effects (font (size 1.27 1.27)) hide)
+    )
+  )
   (symbol (lib_id "Device:R_Small_US") (at 161.29 129.54 90) (unit 1)
     (in_bom yes) (on_board yes)
@@
       (reference "DL1") (unit 1) (value "D_Small") (footprint "00_KeyParts:D_SOD-323_both_sides")
     )
+    (path "/a021078a-949c-459e-b92a-013b035e53ce"
+      (reference "H1") (unit 1) (value "MountingHole") (footprint "00_KeyParts:SpacerHole_M2_4mm")
+    )
+    (path "/2ea98f27-d8a5-41c9-8175-857dfd0bf896"
+      (reference "H2") (unit 1) (value "MountingHole") (footprint "00_KeyParts:SpacerHole_M2_4mm")
+    )
+    (path "/82bb916a-fd01-41e9-abfa-6063b28d2145"
+      (reference "H3") (unit 1) (value "MountingHole") (footprint "00_KeyParts:SpacerHole_M2_4mm")
+    )
+    (path "/df434c24-f13a-4641-99c3-be885e0f943a"
+      (reference "H4") (unit 1) (value "MountingHole") (footprint "00_KeyParts:SpacerHole_M2_4mm")
+    )
+    (path "/92aa456b-f0d2-4f8e-8d14-fa0fa647372e"
+      (reference "H5") (unit 1) (value "MountingHole") (footprint "00_KeyParts:SpacerHole_M2_4mm")
+    )
+    (path "/8309758d-cc18-49e2-ba29-8a3e28e372e9"
+      (reference "H6") (unit 1) (value "MountingHole") (footprint "00_KeyParts:SpacerHole_M2_4mm")
+    )
+    (path "/388a96aa-dab4-4152-8758-f7af6ed35d0e"
+      (reference "H7") (unit 1) (value "MountingHole") (footprint "00_KeyParts:SpacerHole_M2_4mm")
+    )
+    (path "/965bac69-32d3-48c8-a8e7-a928455a03b9"
+      (reference "H8") (unit 1) (value "MountingHole") (footprint "00_KeyParts:SpacerHole_M2_4mm")
+    )
     (path "/afde2c83-3cd9-4387-a068-f4bd55db6222"

Commit message: cap/resister values
Parts:
- C2, C3, C4: value C_Small -> 0.1u
