File: MozzaCircuit/RGB_LED.kicad_sch (KiCad schematic)
At the start: 0 parts

Commit message: led matrix
Parts:
- added C11, C12, C13, C14, C15, C21, C22, C23, C24, C25, C31, C32, C33, C34, C35, C41, C42, C43, C44, C51, C52, C53, C54, C61, C62, C63, C64, C71, C72, C73, C82, C83, C84: C_Small, symbol Device:C_Small
- added L12, L13, L15, L21, L22, L23, L24, L25, L31, L32, L33, L34, L35, L41, L42, L43, L44, L51, L52, L53, L54, L61, L62, L63, L64, L71, L72, L73, L82, L83, L84: WS2812-2020_both_sides, symbol 00_KeyParts:WS2812-2020_both_sides
Connections:
- new net: L24.3 (DIn), L24.7 (DIn), L34.1 (DOut), L34.5 (DOut)
- new net: L34.3 (DIn), L34.7 (DIn), L44.1 (DOut), L44.5 (DOut)
- new net: L83.1 (DOut), L83.5 (DOut), L84.3 (DIn), L84.7 (DIn)
- new net: L73.1 (DOut), L73.5 (DOut), L83.3 (DIn), L83.7 (DIn)
- new net: L44.3 (DIn), L44.7 (DIn), L54.1 (DOut), L54.5 (DOut)
- new net: L54.3 (DIn), L54.7 (DIn), L64.1 (DOut), L64.5 (DOut)
- new net: L52.3 (DIn), L52.7 (DIn), L62.1 (DOut), L62.5 (DOut)
- new net: L62.3 (DIn), L62.7 (DIn), L72.1 (DOut), L72.5 (DOut)
- new net: L43.1 (DOut), L43.5 (DOut), L53.3 (DIn), L53.7 (DIn)
- new net: L33.1 (DOut), L33.5 (DOut), L43.3 (DIn), L43.7 (DIn)
- new net: L35.1 (DOut), L35.5 (DOut)
- new net: L25.1 (DOut), L25.5 (DOut), L35.3 (DIn), L35.7 (DIn)
- new net: L15.1 (DOut), L15.5 (DOut), L25.3 (DIn), L25.7 (DIn)
- new net: L15.3 (DIn), L15.7 (DIn), L24.1 (DOut), L24.5 (DOut)
- new net: L71.1 (DOut), L71.5 (DOut), L82.3 (DIn), L82.7 (DIn)
- new net: L61.1 (DOut), L61.5 (DOut), L71.3 (DIn), L71.7 (DIn)
- new net: L72.3 (DIn), L72.7 (DIn), L82.1 (DOut), L82.5 (DOut)
- new net: L41.1 (DOut), L41.5 (DOut), L51.3 (DIn), L51.7 (DIn)
- new net: L31.1 (DOut), L31.5 (DOut), L41.3 (DIn), L41.7 (DIn)
- new net: L64.3 (DIn), L64.7 (DIn), L84.1 (DOut), L84.5 (DOut)
- new net: L22.3 (DIn), L22.7 (DIn), L32.1 (DOut), L32.5 (DOut)
- new net: L32.3 (DIn), L32.7 (DIn), L42.1 (DOut), L42.5 (DOut)
- new net: L63.1 (DOut), L63.5 (DOut), L73.3 (DIn), L73.7 (DIn)
- new net: L42.3 (DIn), L42.7 (DIn), L52.1 (DOut), L52.5 (DOut)
- new net: L51.1 (DOut), L51.5 (DOut), L61.3 (DIn), L61.7 (DIn)
- new net: L53.1 (DOut), L53.5 (DOut), L63.3 (DIn), L63.7 (DIn)
- new net: L21.1 (DOut), L21.5 (DOut), L31.3 (DIn), L31.7 (DIn)
- new net: L12.3 (DIn), L12.7 (DIn), L22.1 (DOut), L22.5 (DOut)
- new net: L12.1 (DOut), L12.5 (DOut), L13.3 (DIn), L13.7 (DIn)
- new net: L13.1 (DOut), L13.5 (DOut), L23.3 (DIn), L23.7 (DIn)
- new net: L23.1 (DOut), L23.5 (DOut), L33.3 (DIn), L33.7 (DIn)
- new net 5VD: C11.1, C12.1, C13.1, C14.1, C15.1, C21.1, C22.1, C23.1, C24.1, C25.1, C31.1, C32.1, C33.1, C34.1, C35.1, C41.1, C42.1, C43.1, C44.1, C51.1, C52.1, C53.1, C54.1, C61.1, C62.1, C63.1, C64.1, C71.1, C72.1, C73.1, C82.1, C83.1, C84.1, L12.4 (VDD), L12.8, L13.4 (VDD), L13.8, L15.4 (VDD), L15.8, L21.4 (VDD), L21.8, L22.4 (VDD), L22.8, L23.4 (VDD), L23.8, L24.4 (VDD), L24.8, L25.4 (VDD), L25.8, L31.4 (VDD), L31.8, L32.4 (VDD), L32.8, L33.4 (VDD), L33.8, L34.4 (VDD), L34.8, L35.4 (VDD), L35.8, L41.4 (VDD), L41.8, L42.4 (VDD), L42.8, L43.4 (VDD), L43.8, L44.4 (VDD), L44.8, L51.4 (VDD), L51.8, L52.4 (VDD), L52.8, L53.4 (VDD), L53.8, L54.4 (VDD), L54.8, L61.4 (VDD), L61.8, L62.4 (VDD), L62.8, L63.4 (VDD), L63.8, L64.4 (VDD), L64.8, L71.4 (VDD), L71.8, L72.4 (VDD), L72.8, L73.4 (VDD), L73.8, L82.4 (VDD), L82.8, L83.4 (VDD), L83.8, L84.4 (VDD), L84.8
- new net GNDD: C11.2, C12.2, C13.2, C14.2, C15.2, C21.2, C22.2, C23.2, C24.2, C25.2, C31.2, C32.2, C33.2, C34.2, C35.2, C41.2, C42.2, C43.2, C44.2, C51.2, C52.2, C53.2, C54.2, C61.2, C62.2, C63.2, C64.2, C71.2, C72.2, C73.2, C82.2, C83.2, C84.2, L12.2 (GND), L12.6, L13.2 (GND), L13.6, L15.2 (GND), L15.6, L21.2 (GND), L21.6, L22.2 (GND), L22.6, L23.2 (GND), L23.6, L24.2 (GND), L24.6, L25.2 (GND), L25.6, L31.2 (GND), L31.6, L32.2 (GND), L32.6, L33.2 (GND), L33.6, L34.2 (GND), L34.6, L35.2 (GND), L35.6, L41.2 (GND), L41.6, L42.2 (GND), L42.6, L43.2 (GND), L43.6, L44.2 (GND), L44.6, L51.2 (GND), L51.6, L52.2 (GND), L52.6, L53.2 (GND), L53.6, L54.2 (GND), L54.6, L61.2 (GND), L61.6, L62.2 (GND), L62.6, L63.2 (GND), L63.6, L64.2 (GND), L64.6, L71.2 (GND), L71.6, L72.2 (GND), L72.6, L73.2 (GND), L73.6, L82.2 (GND), L82.6, L83.2 (GND), L83.6, L84.2 (GND), L84.6
- new net LED: L21.3 (DIn), L21.7 (DIn)
- no-connect marks 0 -> 1

Commit message: added 3D models, debounce for encoder
Parts:
- C11: value C_Small -> 0.1u; footprint (none) -> 00_KeyParts:C_2012_rev
- C12, C13, C14, C15, C21, C22, C23, C24, C25, C31, C32, C33, C34, C35, C41, C42, C43, C44, C51, C52, C53, C54, C61, C62, C63, C64, C71, C72, C73, C82, C83, C84: footprint (none) -> 00_KeyParts:C_2012_rev
- L12, L13, L15, L21, L22, L23, L24, L25, L31, L32, L33, L34, L35, L41, L42, L43, L44, L51, L52, L53, L54, L61, L62, L63, L64, L71, L72, L73, L82, L83, L84: footprint (none) -> 00_KeyParts:WS2812B_2020_rev

Commit message: started place and route
Parts:
- removed C11: 0.1u, 00_KeyParts:C_2012_rev, symbol Device:C_Small
- removed C14: C_Small, 00_KeyParts:C_2012_rev, symbol Device:C_Small
- added DL1: D_Small, 00_KeyParts:D_SOD-323_both_sides, symbol Device:D_Small
- C21: value C_Small -> 0.1u
Connections:
- net 5VD: now also DL1.2 (A); no longer L21.4 (VDD), L21.8
- new net 4V3D: DL1.1 (K), L21.4 (VDD), L21.8
Changed lines of the file:
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@@
   (junction (at 106.68 74.93) (diameter 0) (color 0 0 0 0)
   )
+  (junction (at 234.95 36.83) (diameter 0) (color 0 0 0 0)
+  )
   (junction (at 86.36 29.21) (diameter 0) (color 0 0 0 0)
   )
-  (junction (at 234.95 36.83) (diameter 0) (color 0 0 0 0)
-  )
   (junction (at 241.3 31.75) (diameter 0) (color 0 0 0 0)
   )
@@
   (junction (at 260.35 74.93) (diameter 0) (color 0 0 0 0)
   )
-  (junction (at 228.6 74.93) (diameter 0) (color 0 0 0 0)
-  )
   (junction (at 127 80.01) (diameter 0) (color 0 0 0 0)
   )
@@
   (junction (at 45.72 130.81) (diameter 0) (color 0 0 0 0)
   )
-  (junction (at 66.04 29.21) (diameter 0) (color 0 0 0 0)
-  )
   (junction (at 106.68 80.01) (diameter 0) (color 0 0 0 0)
   )
@@
   (junction (at 254 62.23) (diameter 0) (color 0 0 0 0)
   )
-  (junction (at 228.6 31.75) (diameter 0) (color 0 0 0 0)
-  )
   (junction (at 86.36 100.33) (diameter 0) (color 0 0 0 0)
   )
@@
   (junction (at 127 29.21) (diameter 0) (color 0 0 0 0)
   )
-  (junction (at 228.6 69.85) (diameter 0) (color 0 0 0 0)
-  )
   (junction (at 66.04 125.73) (diameter 0) (color 0 0 0 0)
   )
@@
   )
   (junction (at 260.35 49.53) (diameter 0) (color 0 0 0 0)
-  )
-  (junction (at 228.6 36.83) (diameter 0) (color 0 0 0 0)
   )
   (junction (at 254 69.85) (diameter 0) (color 0 0 0 0)
@@
     (stroke (width 0) (type default) (color 0 0 0 0))
   )
-  (wire (pts (xy 228.6 74.93) (xy 234.95 74.93))
+  (wire (pts (xy 222.25 74.93) (xy 234.95 74.93))
     (stroke (width 0) (type default) (color 0 0 0 0))
   )
@@
     (stroke (width 0) (type default) (color 0 0 0 0))
   )
-  (wire (pts (xy 222.25 74.93) (xy 228.6 74.93))
-    (stroke (width 0) (type default) (color 0 0 0 0))
-  )
   (wire (pts (xy 86.36 80.01) (xy 106.68 80.01))
     (stroke (width 0) (type default) (color 0 0 0 0))
@@
     (stroke (width 0) (type default) (color 0 0 0 0))
   )
-  (wire (pts (xy 222.25 31.75) (xy 228.6 31.75))
-    (stroke (width 0) (type default) (color 0 0 0 0))
-  )
   (wire (pts (xy 260.35 62.23) (xy 266.7 62.23))
     (stroke (width 0) (type default) (color 0 0 0 0))
@@
     (stroke (width 0) (type default) (color 0 0 0 0))
   )
+  (wire (pts (xy 78.74 29.21) (xy 86.36 29.21))
+    (stroke (width 0) (type default) (color 0 0 0 0))
+  )
   (wire (pts (xy 25.4 74.93) (xy 45.72 74.93))
     (stroke (width 0) (type default) (color 0 0 0 0))
@@
     (stroke (width 0) (type default) (color 0 0 0 0))
   )
-  (wire (pts (xy 228.6 36.83) (xy 234.95 36.83))
-    (stroke (width 0) (type default) (color 0 0 0 0))
-  )
   (wire (pts (xy 127 74.93) (xy 147.32 74.93))
     (stroke (width 0) (type default) (color 0 0 0 0))
@@
     (stroke (width 0) (type default) (color 0 0 0 0))
   )
-  (wire (pts (xy 25.4 29.21) (xy 66.04 29.21))
-    (stroke (width 0) (type default) (color 0 0 0 0))
-  )
   (wire (pts (xy 198.12 90.17) (xy 198.12 115.57))
     (stroke (width 0) (type default) (color 0 0 0 0))
@@
     (stroke (width 0) (type default) (color 0 0 0 0))
   )
-  (wire (pts (xy 66.04 29.21) (xy 86.36 29.21))
-    (stroke (width 0) (type default) (color 0 0 0 0))
-  )
   (wire (pts (xy 66.04 54.61) (xy 86.36 54.61))
     (stroke (width 0) (type default) (color 0 0 0 0))
   )
-  (wire (pts (xy 222.25 69.85) (xy 228.6 69.85))
-    (stroke (width 0) (type default) (color 0 0 0 0))
-  )
   (wire (pts (xy 222.25 87.63) (xy 228.6 87.63))
     (stroke (width 0) (type default) (color 0 0 0 0))
@@
     (stroke (width 0) (type default) (color 0 0 0 0))
   )
-  (wire (pts (xy 228.6 31.75) (xy 234.95 31.75))
+  (wire (pts (xy 222.25 31.75) (xy 234.95 31.75))
     (stroke (width 0) (type default) (color 0 0 0 0))
   )
@@
     (stroke (width 0) (type default) (color 0 0 0 0))
   )
+  (wire (pts (xy 58.42 29.21) (xy 66.04 29.21))
+    (stroke (width 0) (type default) (color 0 0 0 0))
+  )
   (wire (pts (xy 167.64 100.33) (xy 187.96 100.33))
     (stroke (width 0) (type default) (color 0 0 0 0))
@@
     (stroke (width 0) (type default) (color 0 0 0 0))
   )
-  (wire (pts (xy 222.25 36.83) (xy 228.6 36.83))
+  (wire (pts (xy 222.25 36.83) (xy 234.95 36.83))
     (stroke (width 0) (type default) (color 0 0 0 0))
   )
@@
     (stroke (width 0) (type default) (color 0 0 0 0))
   )
-  (wire (pts (xy 228.6 69.85) (xy 234.95 69.85))
-    (stroke (width 0) (type default) (color 0 0 0 0))
-  )
-  (global_label "5VD" (shape input) (at 25.4 29.21 180) (fields_autoplaced)
+  (wire (pts (xy 222.25 69.85) (xy 234.95 69.85))
+    (stroke (width 0) (type default) (color 0 0 0 0))
+  )
+  (global_label "5VD" (shape input) (at 222.25 19.05 180) (fields_autoplaced)
     (effects (font (size 1.27 1.27)) (justify right))
-    (property "Intersheet References" "${INTERSHEET_REFS}" (id 0) (at 19.4188 29.2894 0)
+    (property "Intersheet References" "${INTERSHEET_REFS}" (id 0) (at 216.2688 19.1294 0)
       (effects (font (size 1.27 1.27)) (justify right) hide)
     )
@@
     )
   )
+  (global_label "4V3D" (shape input) (at 227.33 19.05 0) (fields_autoplaced)
+    (effects (font (size 1.27 1.27)) (justify left))
+    (property "Intersheet References" "${INTERSHEET_REFS}" (id 0) (at 234.5207 18.9706 0)
+      (effects (font (size 1.27 1.27)) (justify left) hide)
+    )
+  )
   (global_label "5VD" (shape input) (at 222.25 31.75 180) (fields_autoplaced)
     (effects (font (size 1.27 1.27)) (justify right))
@@
     )
   )
+  (global_label "4V3D" (shape input) (at 247.65 19.05 180) (fields_autoplaced)
+    (effects (font (size 1.27 1.27)) (justify right))
+    (property "Intersheet References" "${INTERSHEET_REFS}" (id 0) (at 240.4593 19.1294 0)
+      (effects (font (size 1.27 1.27)) (justify right) hide)
+    )
+  )
   (global_label "5VD" (shape input) (at 222.25 44.45 180) (fields_autoplaced)
     (effects (font (size 1.27 1.27)) (justify right))
@@
     )
   )
+  (global_label "4V3D" (shape input) (at 58.42 29.21 180) (fields_autoplaced)
+    (effects (font (size 1.27 1.27)) (justify right))
+    (property "Intersheet References" "${INTERSHEET_REFS}" (id 0) (at 51.2293 29.1306 0)
+      (effects (font (size 1.27 1.27)) (justify right) hide)
+    )
+  )
+  (global_label "5VD" (shape input) (at 78.74 29.21 180) (fields_autoplaced)
+    (effects (font (size 1.27 1.27)) (justify right))
+    (property "Intersheet References" "${INTERSHEET_REFS}" (id 0) (at 72.7588 29.2894 0)
+      (effects (font (size 1.27 1.27)) (justify right) hide)
+    )
+  )
   (global_label "5VD" (shape input) (at 25.4 105.41 180) (fields_autoplaced)
     (effects (font (size 1.27 1.27)) (justify right))
@@
       (effects (font (size 1.27 1.27)) (justify left))
     )
-    (property "Value" "C_Small" (id 1) (at 238.125 35.5662 0)
-      (effects (font (size 1.27 1.27)) (justify left) hide)
+    (property "Value" "0.1u" (id 1) (at 233.045 27.94 0)
+      (effects (font (size 1.27 1.27)) (justify left))
     )
     (property "Footprint" "00_KeyParts:C_2012_rev" (id 2) (at 234.95 34.29 0)
@@
     (pin "8")
   )
-  (symbol (lib_id "Device:C_Small") (at 228.6 34.29 0) (unit 1)
-    (in_bom yes) (on_board yes)
-    (property "Reference" "C11" (id 0) (at 227.33 29.845 0)
-      (effects (font (size 1.27 1.27)) (justify left))
-    )
-    (property "Value" "0.1u" (id 1) (at 227.33 27.94 0)
-      (effects (font (size 1.27 1.27)) (justify left))
-    )
-    (property "Footprint" "00_KeyParts:C_2012_rev" (id 2) (at 228.6 34.29 0)
-      (effects (font (size 1.27 1.27)) hide)
-    )
-    (property "Datasheet" "~" (id 3) (at 228.6 34.29 0)
-      (effects (font (size 1.27 1.27)) hide)
-    )
-    (pin "1")
-    (pin "2")
-  )
-  (symbol (lib_id "Device:C_Small") (at 228.6 72.39 0) (unit 1)
-    (in_bom yes) (on_board yes)
-    (property "Reference" "C14" (id 0) (at 227.33 67.945 0)
-      (effects (font (size 1.27 1.27)) (justify left))
-    )
-    (property "Value" "C_Small" (id 1) (at 231.775 73.6662 0)
-      (effects (font (size 1.27 1.27)) (justify left) hide)
-    )
-    (property "Footprint" "00_KeyParts:C_2012_rev" (id 2) (at 228.6 72.39 0)
-      (effects (font (size 1.27 1.27)) hide)
-    )
-    (property "Datasheet" "~" (id 3) (at 228.6 72.39 0)
-      (effects (font (size 1.27 1.27)) hide)
-    )
-    (pin "1")
-    (pin "2")
-  )
   (symbol (lib_id "00_KeyParts:WS2812-2020_both_sides") (at 66.04 90.17 0) (mirror y) (unit 1)
     (in_bom yes) (on_board yes) (fields_autoplaced)
@@
     (pin "8")
   )
+  (symbol (lib_id "Device:D_Small") (at 224.79 19.05 180) (unit 1)
+    (in_bom yes) (on_board yes) (fields_autoplaced)
+    (property "Reference" "DL1" (id 0) (at 224.79 15.875 0))
+    (property "Value" "D_Small" (id 1) (at 224.79 15.875 0)
+      (effects (font (size 1.27 1.27)) hide)
+    )
+    (property "Footprint" "00_KeyParts:D_SOD-323_both_sides" (id 2) (at 224.79 19.05 90)
+      (effects (font (size 1.27 1.27)) hide)
+    )
+    (property "Datasheet" "~" (id 3) (at 224.79 19.05 90)
+      (effects (font (size 1.27 1.27)) hide)
+    )
+    (pin "1")
+    (pin "2")
+  )
   (symbol (lib_id "power:GNDD") (at 222.25 74.93 270) (unit 1)
     (in_bom yes) (on_board yes) (fields_autoplaced)
@@
       (effects (font (size 1.27 1.27)) hide)
     )
+    (pin "1")
+  )
+  (symbol (lib_id "power:PWR_FLAG") (at 247.65 19.05 270) (unit 1)
+    (in_bom yes) (on_board yes) (fields_autoplaced)
+    (property "Reference" "#FLG0105" (id 0) (at 249.555 19.05 0)
+      (effects (font (size 1.27 1.27)) hide)
+    )
+    (property "Value" "PWR_FLAG" (id 1) (at 250.825 19.0499 90)
+      (effects (font (size 1.27 1.27)) (justify left))
+    )
+    (property "Footprint" "" (id 2) (at 247.65 19.05 0)
+      (effects (font (size 1.27 1.27)) hide)
+    )
+    (property "Datasheet" "~" (id 3) (at 247.65 19.05 0)
+      (effects (font (size 1.27 1.27)) hide)
+    )

Commit message: led direction
Parts:
- renumbered C12 to C14, L12 to L14
Connections:
- net at L15.3 (DIn), L15.7 (DIn): now also L14.1 (DOut), L14.5 (DOut); no longer L24.1 (DOut), L24.5 (DOut)
- net at L22.1 (DOut), L22.5 (DOut): now also L13.3 (DIn), L13.7 (DIn); no longer L14.3 (DIn), L14.7 (DIn)
- new net: L14.3 (DIn), L14.7 (DIn), L24.1 (DOut), L24.5 (DOut)
Other:
- moved on the sheet: C14, L14
Changed lines of the file:
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@@
   (junction (at 234.95 87.63) (diameter 0) (color 0 0 0 0)
   )
-  (junction (at 228.6 44.45) (diameter 0) (color 0 0 0 0)
-  )
   (junction (at 234.95 62.23) (diameter 0) (color 0 0 0 0)
   )
@@
   (junction (at 127 49.53) (diameter 0) (color 0 0 0 0)
   )
-  (junction (at 45.72 54.61) (diameter 0) (color 0 0 0 0)
-  )
   (junction (at 247.65 74.93) (diameter 0) (color 0 0 0 0)
   )
@@
   (junction (at 266.7 44.45) (diameter 0) (color 0 0 0 0)
   )
-  (junction (at 228.6 49.53) (diameter 0) (color 0 0 0 0)
-  )
   (junction (at 167.64 74.93) (diameter 0) (color 0 0 0 0)
   )
@@
   (junction (at 228.6 82.55) (diameter 0) (color 0 0 0 0)
   )
+  (junction (at 228.6 69.85) (diameter 0) (color 0 0 0 0)
+  )
   (junction (at 260.35 74.93) (diameter 0) (color 0 0 0 0)
   )
@@
   (junction (at 167.64 80.01) (diameter 0) (color 0 0 0 0)
   )
-  (junction (at 45.72 74.93) (diameter 0) (color 0 0 0 0)
+  (junction (at 228.6 74.93) (diameter 0) (color 0 0 0 0)
   )
   (junction (at 147.32 49.53) (diameter 0) (color 0 0 0 0)
@@
   )
   (junction (at 147.32 105.41) (diameter 0) (color 0 0 0 0)
+  )
+  (junction (at 45.72 125.73) (diameter 0) (color 0 0 0 0)
+  )
+  (junction (at 45.72 105.41) (diameter 0) (color 0 0 0 0)
   )
   (junction (at 127 100.33) (diameter 0) (color 0 0 0 0)
@@
     (stroke (width 0) (type default) (color 0 0 0 0))
   )
-  (wire (pts (xy 25.4 105.41) (xy 66.04 105.41))
+  (wire (pts (xy 25.4 105.41) (xy 45.72 105.41))
     (stroke (width 0) (type default) (color 0 0 0 0))
   )
@@
     (stroke (width 0) (type default) (color 0 0 0 0))
   )
-  (wire (pts (xy 25.4 54.61) (xy 45.72 54.61))
-    (stroke (width 0) (type default) (color 0 0 0 0))
-  )
   (wire (pts (xy 127 80.01) (xy 147.32 80.01))
     (stroke (width 0) (type default) (color 0 0 0 0))
   )
-  (wire (pts (xy 25.4 125.73) (xy 66.04 125.73))
+  (wire (pts (xy 45.72 105.41) (xy 66.04 105.41))
+    (stroke (width 0) (type default) (color 0 0 0 0))
+  )
+  (wire (pts (xy 25.4 125.73) (xy 45.72 125.73))
     (stroke (width 0) (type default) (color 0 0 0 0))
   )
@@
     (stroke (width 0) (type default) (color 0 0 0 0))
   )
-  (wire (pts (xy 222.25 74.93) (xy 234.95 74.93))
+  (wire (pts (xy 222.25 74.93) (xy 228.6 74.93))
     (stroke (width 0) (type default) (color 0 0 0 0))
   )
@@
     (stroke (width 0) (type default) (color 0 0 0 0))
   )
-  (wire (pts (xy 222.25 49.53) (xy 228.6 49.53))
-    (stroke (width 0) (type default) (color 0 0 0 0))
-  )
   (wire (pts (xy 241.3 36.83) (xy 247.65 36.83))
     (stroke (width 0) (type default) (color 0 0 0 0))
@@
     (stroke (width 0) (type default) (color 0 0 0 0))
   )
-  (wire (pts (xy 228.6 49.53) (xy 234.95 49.53))
+  (wire (pts (xy 222.25 49.53) (xy 234.95 49.53))
     (stroke (width 0) (type default) (color 0 0 0 0))
   )
@@
     (stroke (width 0) (type default) (color 0 0 0 0))
   )
-  (wire (pts (xy 25.4 74.93) (xy 45.72 74.93))
-    (stroke (width 0) (type default) (color 0 0 0 0))
-  )
   (wire (pts (xy 66.04 151.13) (xy 86.36 151.13))
     (stroke (width 0) (type default) (color 0 0 0 0))
   )
+  (wire (pts (xy 35.56 64.77) (xy 55.88 64.77))
+    (stroke (width 0) (type default) (color 0 0 0 0))
+  )
   (wire (pts (xy 86.36 100.33) (xy 106.68 100.33))
     (stroke (width 0) (type default) (color 0 0 0 0))
@@
     (stroke (width 0) (type default) (color 0 0 0 0))
   )
-  (wire (pts (xy 45.72 74.93) (xy 66.04 74.93))
+  (wire (pts (xy 25.4 74.93) (xy 66.04 74.93))
     (stroke (width 0) (type default) (color 0 0 0 0))
   )
@@
     (stroke (width 0) (type default) (color 0 0 0 0))
   )
-  (wire (pts (xy 45.72 54.61) (xy 66.04 54.61))
+  (wire (pts (xy 25.4 54.61) (xy 66.04 54.61))
     (stroke (width 0) (type default) (color 0 0 0 0))
   )
@@
     (stroke (width 0) (type default) (color 0 0 0 0))
   )
-  (wire (pts (xy 228.6 44.45) (xy 234.95 44.45))
+  (wire (pts (xy 222.25 44.45) (xy 234.95 44.45))
     (stroke (width 0) (type default) (color 0 0 0 0))
   )
@@
     (stroke (width 0) (type default) (color 0 0 0 0))
   )
+  (wire (pts (xy 228.6 74.93) (xy 234.95 74.93))
+    (stroke (width 0) (type default) (color 0 0 0 0))
+  )
   (wire (pts (xy 241.3 74.93) (xy 247.65 74.93))
     (stroke (width 0) (type default) (color 0 0 0 0))
@@
     (stroke (width 0) (type default) (color 0 0 0 0))
   )
+  (wire (pts (xy 45.72 125.73) (xy 66.04 125.73))
+    (stroke (width 0) (type default) (color 0 0 0 0))
+  )
   (wire (pts (xy 228.6 87.63) (xy 234.95 87.63))
     (stroke (width 0) (type default) (color 0 0 0 0))
@@
     (stroke (width 0) (type default) (color 0 0 0 0))
   )
-  (wire (pts (xy 55.88 115.57) (xy 35.56 115.57))
-    (stroke (width 0) (type default) (color 0 0 0 0))
-  )
   (wire (pts (xy 157.48 115.57) (xy 177.8 115.57))
     (stroke (width 0) (type default) (color 0 0 0 0))
@@
     (stroke (width 0) (type default) (color 0 0 0 0))
   )
-  (wire (pts (xy 222.25 44.45) (xy 228.6 44.45))
+  (wire (pts (xy 228.6 69.85) (xy 234.95 69.85))
     (stroke (width 0) (type default) (color 0 0 0 0))
   )
@@
     (stroke (width 0) (type default) (color 0 0 0 0))
   )
-  (wire (pts (xy 222.25 69.85) (xy 234.95 69.85))
+  (wire (pts (xy 222.25 69.85) (xy 228.6 69.85))
     (stroke (width 0) (type default) (color 0 0 0 0))
   )
@@
     (pin "8")
   )
-  (symbol (lib_id "Device:C_Small") (at 228.6 46.99 0) (unit 1)
-    (in_bom yes) (on_board yes)
-    (property "Reference" "C12" (id 0) (at 227.33 42.545 0)
-      (effects (font (size 1.27 1.27)) (justify left))
-    )
-    (property "Value" "C_Small" (id 1) (at 231.775 48.2662 0)
-      (effects (font (size 1.27 1.27)) (justify left) hide)
-    )
-    (property "Footprint" "00_KeyParts:C_2012_rev" (id 2) (at 228.6 46.99 0)
-      (effects (font (size 1.27 1.27)) hide)
-    )
-    (property "Datasheet" "~" (id 3) (at 228.6 46.99 0)
+  (symbol (lib_id "Device:C_Small") (at 228.6 72.39 0) (unit 1)
+    (in_bom yes) (on_board yes)
+    (property "Reference" "C14" (id 0) (at 227.33 67.945 0)
+      (effects (font (size 1.27 1.27)) (justify left))
+    )
+    (property "Value" "C_Small" (id 1) (at 231.775 73.6662 0)
+      (effects (font (size 1.27 1.27)) (justify left) hide)
+    )
+    (property "Footprint" "00_KeyParts:C_2012_rev" (id 2) (at 228.6 72.39 0)
+      (effects (font (size 1.27 1.27)) hide)
+    )
+    (property "Datasheet" "~" (id 3) (at 228.6 72.39 0)
       (effects (font (size 1.27 1.27)) hide)
     )
@@
     (pin "2")
   )
-  (symbol (lib_id "00_KeyParts:WS2812-2020_both_sides") (at 45.72 64.77 0) (unit 1)
-    (in_bom yes) (on_board yes)
-    (property "Reference" "L12" (id 0) (at 55.88 60.96 0))
-    (property "Value" "WS2812-2020_both_sides" (id 1) (at 58.42 73.66 0)
-      (effects (font (size 1.016 1.016)) hide)
-    )
-    (property "Footprint" "00_KeyParts:WS2812B_2020_rev" (id 2) (at 45.72 64.77 0)
-      (effects (font (size 1.524 1.524)) hide)
-    )
-    (property "Datasheet" "" (id 3) (at 45.72 64.77 0)
-      (effects (font (size 1.524 1.524)) hide)
-    )
+  (symbol (lib_id "00_KeyParts:WS2812-2020_both_sides") (at 45.72 115.57 0) (unit 1)
+    (in_bom yes) (on_board yes)
+    (property "Reference" "L14" (id 0) (at 55.88 111.76 0))
+    (property "Value" "WS2812-2020_both_sides" (id 1) (at 58.42 124.46 0)
+      (effects (font (size 1.016 1.016)) hide)
+    )
+    (property "Footprint" "00_KeyParts:WS2812B_2020_rev" (id 2) (at 45.72 115.57 0)
+      (effects (font (size 1.524 1.524)) hide)
+    )
+    (property "Datasheet" "" (id 3) (at 45.72 115.57 0)
+      (effects (font (size 1.524 1.524)) hide)
+    )

Commit message: 1608 R&C
Parts:
- C13, C14, C15, C21, C22, C23, C24, C25, C31, C32, C33, C34, C35, C41, C42, C43, C44, C51, C52, C53, C54, C61, C62, C63, C64, C71, C72, C73, C82, C83, C84: footprint 00_KeyParts:C_2012_rev -> 00_KeyParts:C_1608_HandSolder_both_sides
Connections:
- net 4V3D: now also C21.1
- net 5VD: no longer C21.1
