File: MozzaCircuit/RGB_LED.kicad_sch (KiCad schematic)
At the start: 63 parts

Commit message: cap/resister values
Parts:
- C13, C14, C15, C22, C23, C24, C25, C31, C32, C33, C34, C35, C41, C42, C43, C44, C51, C52, C53, C54, C61, C62, C63, C64, C71, C72, C73, C82, C83, C84: value C_Small -> 0.1u
Changed lines of the file:
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@@
       (effects (font (size 1.27 1.27)) (justify left))
     )
-    (property "Value" "C_Small" (id 1) (at 250.825 35.5662 0)
+    (property "Value" "0.1u" (id 1) (at 250.825 35.5662 0)
       (effects (font (size 1.27 1.27)) (justify left) hide)
     )
@@
       (effects (font (size 1.27 1.27)) (justify left))
     )
-    (property "Value" "C_Small" (id 1) (at 244.475 60.9662 0)
+    (property "Value" "0.1u" (id 1) (at 244.475 60.9662 0)
       (effects (font (size 1.27 1.27)) (justify left) hide)
     )
@@
       (effects (font (size 1.27 1.27)) (justify left))
     )
-    (property "Value" "C_Small" (id 1) (at 269.875 48.2662 0)
+    (property "Value" "0.1u" (id 1) (at 269.875 48.2662 0)
       (effects (font (size 1.27 1.27)) (justify left) hide)
     )
@@
       (effects (font (size 1.27 1.27)) (justify left))
     )
-    (property "Value" "C_Small" (id 1) (at 257.175 73.6662 0)
+    (property "Value" "0.1u" (id 1) (at 257.175 73.6662 0)
       (effects (font (size 1.27 1.27)) (justify left) hide)
     )
@@
       (effects (font (size 1.27 1.27)) (justify left))
     )
-    (property "Value" "C_Small" (id 1) (at 250.825 73.6662 0)
+    (property "Value" "0.1u" (id 1) (at 250.825 73.6662 0)
       (effects (font (size 1.27 1.27)) (justify left) hide)
     )
@@
       (effects (font (size 1.27 1.27)) (justify left))
     )
-    (property "Value" "C_Small" (id 1) (at 250.825 60.9662 0)
+    (property "Value" "0.1u" (id 1) (at 250.825 60.9662 0)
       (effects (font (size 1.27 1.27)) (justify left) hide)
     )
@@
       (effects (font (size 1.27 1.27)) (justify left))
     )
-    (property "Value" "C_Small" (id 1) (at 231.775 73.6662 0)
+    (property "Value" "0.1u" (id 1) (at 231.775 73.6662 0)
       (effects (font (size 1.27 1.27)) (justify left) hide)
     )
@@
       (effects (font (size 1.27 1.27)) (justify left))
     )
-    (property "Value" "C_Small" (id 1) (at 238.125 48.2662 0)
+    (property "Value" "0.1u" (id 1) (at 238.125 48.2662 0)
       (effects (font (size 1.27 1.27)) (justify left) hide)
     )
@@
       (effects (font (size 1.27 1.27)) (justify left))
     )
-    (property "Value" "C_Small" (id 1) (at 263.525 60.9662 0)
+    (property "Value" "0.1u" (id 1) (at 263.525 60.9662 0)
       (effects (font (size 1.27 1.27)) (justify left) hide)
     )
@@
       (effects (font (size 1.27 1.27)) (justify left))
     )
-    (property "Value" "C_Small" (id 1) (at 238.125 86.3662 0)
+    (property "Value" "0.1u" (id 1) (at 238.125 86.3662 0)
       (effects (font (size 1.27 1.27)) (justify left) hide)
     )
@@
       (effects (font (size 1.27 1.27)) (justify left))
     )
-    (property "Value" "C_Small" (id 1) (at 276.225 60.9662 0)
+    (property "Value" "0.1u" (id 1) (at 276.225 60.9662 0)
       (effects (font (size 1.27 1.27)) (justify left) hide)
     )
@@
       (effects (font (size 1.27 1.27)) (justify left))
     )
-    (property "Value" "C_Small" (id 1) (at 231.775 86.3662 0)
+    (property "Value" "0.1u" (id 1) (at 231.775 86.3662 0)
       (effects (font (size 1.27 1.27)) (justify left) hide)
     )
@@
       (effects (font (size 1.27 1.27)) (justify left))
     )
-    (property "Value" "C_Small" (id 1) (at 244.475 73.6662 0)
+    (property "Value" "0.1u" (id 1) (at 244.475 73.6662 0)
       (effects (font (size 1.27 1.27)) (justify left) hide)
     )
@@
       (effects (font (size 1.27 1.27)) (justify left))
     )
-    (property "Value" "C_Small" (id 1) (at 263.525 73.6662 0)
+    (property "Value" "0.1u" (id 1) (at 263.525 73.6662 0)
       (effects (font (size 1.27 1.27)) (justify left) hide)
     )
@@
       (effects (font (size 1.27 1.27)) (justify left))
     )
-    (property "Value" "C_Small" (id 1) (at 250.825 48.2662 0)
+    (property "Value" "0.1u" (id 1) (at 250.825 48.2662 0)
       (effects (font (size 1.27 1.27)) (justify left) hide)
     )
@@
       (effects (font (size 1.27 1.27)) (justify left))
     )
-    (property "Value" "C_Small" (id 1) (at 238.125 73.6662 0)
+    (property "Value" "0.1u" (id 1) (at 238.125 73.6662 0)
       (effects (font (size 1.27 1.27)) (justify left) hide)
     )
@@
       (effects (font (size 1.27 1.27)) (justify left))
     )
-    (property "Value" "C_Small" (id 1) (at 269.875 60.9662 0)
+    (property "Value" "0.1u" (id 1) (at 269.875 60.9662 0)
       (effects (font (size 1.27 1.27)) (justify left) hide)
     )
@@
       (effects (font (size 1.27 1.27)) (justify left))
     )
-    (property "Value" "C_Small" (id 1) (at 257.175 48.2662 0)
+    (property "Value" "0.1u" (id 1) (at 257.175 48.2662 0)
       (effects (font (size 1.27 1.27)) (justify left) hide)
     )
@@
       (effects (font (size 1.27 1.27)) (justify left))
     )
-    (property "Value" "C_Small" (id 1) (at 244.475 35.5662 0)
+    (property "Value" "0.1u" (id 1) (at 244.475 35.5662 0)
       (effects (font (size 1.27 1.27)) (justify left) hide)
     )
@@
       (effects (font (size 1.27 1.27)) (justify left))
     )
-    (property "Value" "C_Small" (id 1) (at 263.525 48.2662 0)
+    (property "Value" "0.1u" (id 1) (at 263.525 48.2662 0)
       (effects (font (size 1.27 1.27)) (justify left) hide)
     )
@@
       (effects (font (size 1.27 1.27)) (justify left))
     )
-    (property "Value" "C_Small" (id 1) (at 276.225 48.2662 0)
+    (property "Value" "0.1u" (id 1) (at 276.225 48.2662 0)
       (effects (font (size 1.27 1.27)) (justify left) hide)
     )
@@
       (effects (font (size 1.27 1.27)) (justify left))
     )
-    (property "Value" "C_Small" (id 1) (at 238.125 60.9662 0)
+    (property "Value" "0.1u" (id 1) (at 238.125 60.9662 0)
       (effects (font (size 1.27 1.27)) (justify left) hide)
     )
@@
       (effects (font (size 1.27 1.27)) (justify left))
     )
-    (property "Value" "C_Small" (id 1) (at 244.475 48.2662 0)
+    (property "Value" "0.1u" (id 1) (at 244.475 48.2662 0)
       (effects (font (size 1.27 1.27)) (justify left) hide)
     )
@@
       (effects (font (size 1.27 1.27)) (justify left))
     )
-    (property "Value" "C_Small" (id 1) (at 263.525 35.5662 0)
+    (property "Value" "0.1u" (id 1) (at 263.525 35.5662 0)
       (effects (font (size 1.27 1.27)) (justify left) hide)
     )
@@
       (effects (font (size 1.27 1.27)) (justify left))
     )
-    (property "Value" "C_Small" (id 1) (at 276.225 73.6662 0)
+    (property "Value" "0.1u" (id 1) (at 276.225 73.6662 0)
       (effects (font (size 1.27 1.27)) (justify left) hide)
     )
@@
       (effects (font (size 1.27 1.27)) (justify left))
     )
-    (property "Value" "C_Small" (id 1) (at 244.475 86.3662 0)
+    (property "Value" "0.1u" (id 1) (at 244.475 86.3662 0)
       (effects (font (size 1.27 1.27)) (justify left) hide)
     )
@@
       (effects (font (size 1.27 1.27)) (justify left))
     )
-    (property "Value" "C_Small" (id 1) (at 231.775 60.9662 0)
+    (property "Value" "0.1u" (id 1) (at 231.775 60.9662 0)
       (effects (font (size 1.27 1.27)) (justify left) hide)
     )
@@
       (effects (font (size 1.27 1.27)) (justify left))
     )
-    (property "Value" "C_Small" (id 1) (at 257.175 60.9662 0)
+    (property "Value" "0.1u" (id 1) (at 257.175 60.9662 0)
       (effects (font (size 1.27 1.27)) (justify left) hide)
     )
@@
       (effects (font (size 1.27 1.27)) (justify left))
     )
-    (property "Value" "C_Small" (id 1) (at 269.875 35.5662 0)
+    (property "Value" "0.1u" (id 1) (at 269.875 35.5662 0)
       (effects (font (size 1.27 1.27)) (justify left) hide)
     )
@@
       (effects (font (size 1.27 1.27)) (justify left))
     )
-    (property "Value" "C_Small" (id 1) (at 257.175 35.5662 0)
-      (effects (font (size 1.27 1.27)) (justify left) hide)
-    )
+    (property "Value" "0.1u" (id 1) (at 257.175 35.5662 0)
+      (effects (font (size 1.27 1.27)) (justify left) hide)
+    )
