File: MozzaBottom/MozzaBottom.kicad_sch (KiCad schematic)
At the start: 8 parts

Commit message: trying rule areas
Parts:
- added P1: DummyPad, 00_KeyParts:DummyPad, symbol 00_KeyParts:DummyPad
Connections:
- net GND: now also P1.1
Changed lines of the file:
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@@
     )
+  )
+  (symbol (lib_id "power:GND") (at 44.45 38.1 0) (unit 1)
+    (in_bom yes) (on_board yes) (fields_autoplaced)
+    (property "Reference" "#PWR0102" (id 0) (at 44.45 44.45 0)
+      (effects (font (size 1.27 1.27)) hide)
+    )
+    (property "Value" "GND" (id 1) (at 44.45 42.545 0))
+    (property "Footprint" "" (id 2) (at 44.45 38.1 0)
+      (effects (font (size 1.27 1.27)) hide)
+    )
+    (property "Datasheet" "" (id 3) (at 44.45 38.1 0)
+      (effects (font (size 1.27 1.27)) hide)
+    )
+    (pin "1")
   )
   (symbol (lib_id "Mechanical:MountingHole") (at 82.55 57.15 0) (unit 1)
@@
     )
     (property "Datasheet" "~" (id 3) (at 38.1 38.1 0)
+      (effects (font (size 1.27 1.27)) hide)
+    )
+    (pin "1")
+  )
+  (symbol (lib_id "00_KeyParts:DummyPad") (at 41.91 38.1 90) (unit 1)
+    (in_bom yes) (on_board yes) (fields_autoplaced)
+    (property "Reference" "P1" (id 0) (at 46.99 33.0199 90)
+      (effects (font (size 1.27 1.27)) (justify right))
+    )
+    (property "Value" "DummyPad" (id 1) (at 46.99 35.5599 90)
+      (effects (font (size 1.27 1.27)) (justify right))
+    )
+    (property "Footprint" "00_KeyParts:DummyPad" (id 2) (at 41.91 38.1 0)
+      (effects (font (size 1.27 1.27)) hide)
+    )
+    (property "Datasheet" "" (id 3) (at 41.91 38.1 0)
       (effects (font (size 1.27 1.27)) hide)
     )
@@
       (reference "#PWR0101") (unit 1) (value "GND") (footprint "")
     )
+    (path "/56859bb3-2003-461b-876c-5c37497f823d"
+      (reference "#PWR0102") (unit 1) (value "GND") (footprint "")
+    )
     (path "/cbf92050-a678-4199-9407-2ece198d2f6e"
       (reference "H1") (unit 1) (value "MountingHole") (footprint "00_KeyParts:MountingHole_2.3mm_M2")
@@
       (reference "H8") (unit 1) (value "MountingHole") (footprint "00_KeyParts:MountingHole_2.3mm_M2")
     )
+    (path "/b9f33978-5f6c-446e-a1f7-406df70e8587"
+      (reference "P1") (unit 1) (value "DummyPad") (footprint "00_KeyParts:DummyPad")
+    )
   )

Commit message: back side
Parts:
- added P2: DummyPad, 00_KeyParts:DummyPad, symbol 00_KeyParts:DummyPad
Connections:
- net GND: now also P2.1
Changed lines of the file:
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@@
     )
+  )
+  (symbol (lib_id "00_KeyParts:DummyPad") (at 48.26 38.1 90) (unit 1)
+    (in_bom yes) (on_board yes)
+    (property "Reference" "P2" (id 0) (at 49.53 31.115 90)
+      (effects (font (size 1.27 1.27)) (justify right))
+    )
+    (property "Value" "DummyPad" (id 1) (at 53.34 35.5599 90)
+      (effects (font (size 1.27 1.27)) (justify right) hide)
+    )
+    (property "Footprint" "00_KeyParts:DummyPad" (id 2) (at 48.26 38.1 0)
+      (effects (font (size 1.27 1.27)) hide)
+    )
+    (property "Datasheet" "" (id 3) (at 48.26 38.1 0)
+      (effects (font (size 1.27 1.27)) hide)
+    )
+    (pin "1")
   )
   (symbol (lib_id "Mechanical:MountingHole") (at 63.5 57.15 0) (unit 1)
@@
     (pin "1")
   )
+  (symbol (lib_id "power:GND") (at 50.8 38.1 0) (unit 1)
+    (in_bom yes) (on_board yes) (fields_autoplaced)
+    (property "Reference" "#PWR0103" (id 0) (at 50.8 44.45 0)
+      (effects (font (size 1.27 1.27)) hide)
+    )
+    (property "Value" "GND" (id 1) (at 50.8 42.545 0))
+    (property "Footprint" "" (id 2) (at 50.8 38.1 0)
+      (effects (font (size 1.27 1.27)) hide)
+    )
+    (property "Datasheet" "" (id 3) (at 50.8 38.1 0)
+      (effects (font (size 1.27 1.27)) hide)
+    )
+    (pin "1")
+  )
   (symbol (lib_id "Mechanical:MountingHole") (at 82.55 57.15 0) (unit 1)
     (in_bom yes) (on_board yes) (fields_autoplaced)
@@
   )
   (symbol (lib_id "00_KeyParts:DummyPad") (at 41.91 38.1 90) (unit 1)
-    (in_bom yes) (on_board yes) (fields_autoplaced)
-    (property "Reference" "P1" (id 0) (at 46.99 33.0199 90)
+    (in_bom yes) (on_board yes)
+    (property "Reference" "P1" (id 0) (at 43.18 31.115 90)
       (effects (font (size 1.27 1.27)) (justify right))
     )
     (property "Value" "DummyPad" (id 1) (at 46.99 35.5599 90)
-      (effects (font (size 1.27 1.27)) (justify right))
+      (effects (font (size 1.27 1.27)) (justify right) hide)
     )
     (property "Footprint" "00_KeyParts:DummyPad" (id 2) (at 41.91 38.1 0)
@@
       (reference "#PWR0102") (unit 1) (value "GND") (footprint "")
     )
+    (path "/7791f4bd-0884-49dd-bc29-ca70005e6aac"
+      (reference "#PWR0103") (unit 1) (value "GND") (footprint "")
+    )
     (path "/cbf92050-a678-4199-9407-2ece198d2f6e"
       (reference "H1") (unit 1) (value "MountingHole") (footprint "00_KeyParts:MountingHole_2.3mm_M2")
@@
       (reference "P1") (unit 1) (value "DummyPad") (footprint "00_KeyParts:DummyPad")
     )
-  )
+    (path "/1193fe83-61c0-4976-aba8-233f45f0699b"
+      (reference "P2") (unit 1) (value "DummyPad") (footprint "00_KeyParts:DummyPad")
+    )
+  )
