File: Mozzarella/Mozzarella.kicad_sch (KiCad schematic)
At the start: 11 parts, among them J1 RJ45_LED_Shielded_x2, J3 Conn_01x07, J4 Conn_01x07, U1 SeeeduinoXIAO

Commit message: add caps
Parts:
- removed H1: MountingHole, MountingHole:MountingHole_2.2mm_M2, symbol Mechanical:MountingHole
- added C1, C2: 0.1u, 00_KeyParts:C_1608_HandSolder, symbol Device:C_Small
Connections:
- net 3V3: now also C2.1
- net 5VD: now also C1.2
- net GND: now also C1.1, C2.2
Changed lines of the file:
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@@
+    )
+  )
+  (global_label "5VD" (shape input) (at 31.75 131.445 90) (fields_autoplaced)
+    (effects (font (size 1.27 1.27)) (justify left))
+    (property "Intersheet References" "${INTERSHEET_REFS}" (id 0) (at 31.6706 125.4638 90)
+      (effects (font (size 1.27 1.27)) (justify left) hide)
     )
   )
@@
     )
   )
+  (global_label "3V3" (shape input) (at 38.1 131.445 90) (fields_autoplaced)
+    (effects (font (size 1.27 1.27)) (justify left))
+    (property "Intersheet References" "${INTERSHEET_REFS}" (id 0) (at 38.0206 125.5243 90)
+      (effects (font (size 1.27 1.27)) (justify left) hide)
+    )
+  )
+  (global_label "SCK" (shape input) (at 31.115 109.22 180) (fields_autoplaced)
+    (effects (font (size 1.27 1.27)) (justify right))
+    (property "Intersheet References" "${INTERSHEET_REFS}" (id 0) (at 24.9524 109.2994 0)
+      (effects (font (size 1.27 1.27)) (justify right) hide)
+    )
+  )
+  (global_label "3V3" (shape input) (at 114.3 81.28 0) (fields_autoplaced)
+    (effects (font (size 1.27 1.27)) (justify left))
+    (property "Intersheet References" "${INTERSHEET_REFS}" (id 0) (at 120.2207 81.2006 0)
+      (effects (font (size 1.27 1.27)) (justify left) hide)
+    )
+  )
+  (global_label "RGB2" (shape input) (at 88.9 81.28 180) (fields_autoplaced)
+    (effects (font (size 1.27 1.27)) (justify right))
+    (property "Intersheet References" "${INTERSHEET_REFS}" (id 0) (at 81.4674 81.2006 0)
+      (effects (font (size 1.27 1.27)) (justify right) hide)
+    )
+  )
+  (global_label "NRST" (shape input) (at 63.5 71.12 0) (fields_autoplaced)
+    (effects (font (size 1.27 1.27)) (justify left))
+    (property "Intersheet References" "${INTERSHEET_REFS}" (id 0) (at 70.6907 71.0406 0)
+      (effects (font (size 1.27 1.27)) (justify left) hide)
+    )
+  )
+  (global_label "SCK" (shape input) (at 63.5 76.2 0) (fields_autoplaced)
+    (effects (font (size 1.27 1.27)) (justify left))
+    (property "Intersheet References" "${INTERSHEET_REFS}" (id 0) (at 69.6626 76.1206 0)
+      (effects (font (size 1.27 1.27)) (justify left) hide)
+    )
+  )
   (global_label "3V3" (shape input) (at 63.5 146.05 90) (fields_autoplaced)
     (effects (font (size 1.27 1.27)) (justify left))
     (property "Intersheet References" "${INTERSHEET_REFS}" (id 0) (at 63.4206 140.1293 90)
-      (effects (font (size 1.27 1.27)) (justify left) hide)
-    )
-  )
-  (global_label "SCK" (shape input) (at 31.115 109.22 180) (fields_autoplaced)
-    (effects (font (size 1.27 1.27)) (justify right))
-    (property "Intersheet References" "${INTERSHEET_REFS}" (id 0) (at 24.9524 109.2994 0)
-      (effects (font (size 1.27 1.27)) (justify right) hide)
-    )
-  )
-  (global_label "3V3" (shape input) (at 114.3 81.28 0) (fields_autoplaced)
-    (effects (font (size 1.27 1.27)) (justify left))
-    (property "Intersheet References" "${INTERSHEET_REFS}" (id 0) (at 120.2207 81.2006 0)
-      (effects (font (size 1.27 1.27)) (justify left) hide)
-    )
-  )
-  (global_label "RGB2" (shape input) (at 88.9 81.28 180) (fields_autoplaced)
-    (effects (font (size 1.27 1.27)) (justify right))
-    (property "Intersheet References" "${INTERSHEET_REFS}" (id 0) (at 81.4674 81.2006 0)
-      (effects (font (size 1.27 1.27)) (justify right) hide)
-    )
-  )
-  (global_label "NRST" (shape input) (at 63.5 71.12 0) (fields_autoplaced)
-    (effects (font (size 1.27 1.27)) (justify left))
-    (property "Intersheet References" "${INTERSHEET_REFS}" (id 0) (at 70.6907 71.0406 0)
-      (effects (font (size 1.27 1.27)) (justify left) hide)
-    )
-  )
-  (global_label "SCK" (shape input) (at 63.5 76.2 0) (fields_autoplaced)
-    (effects (font (size 1.27 1.27)) (justify left))
-    (property "Intersheet References" "${INTERSHEET_REFS}" (id 0) (at 69.6626 76.1206 0)
       (effects (font (size 1.27 1.27)) (justify left) hide)
     )
@@
     )
     (property "Datasheet" "" (id 3) (at 63.5 63.5 0)
+      (effects (font (size 1.27 1.27)) hide)
+    )
+    (pin "1")
+  )
+  (symbol (lib_id "power:GND") (at 31.75 136.525 0) (unit 1)
+    (in_bom yes) (on_board yes)
+    (property "Reference" "#PWR0102" (id 0) (at 31.75 142.875 0)
+      (effects (font (size 1.27 1.27)) hide)
+    )
+    (property "Value" "GND" (id 1) (at 31.75 144.145 90)
+      (effects (font (size 1.27 1.27)) (justify left))
+    )
+    (property "Footprint" "" (id 2) (at 31.75 136.525 0)
+      (effects (font (size 1.27 1.27)) hide)
+    )
+    (property "Datasheet" "" (id 3) (at 31.75 136.525 0)
       (effects (font (size 1.27 1.27)) hide)
     )
@@
   )
   (symbol (lib_id "Seeeduino XIAO:SeeeduinoXIAO") (at 76.2 109.22 0) (unit 1)
-    (in_bom yes) (on_board no) (fields_autoplaced)
+    (in_bom yes) (on_board yes) (fields_autoplaced)
     (property "Reference" "U1" (id 0) (at 80.7594 130.81 0)
       (effects (font (size 1.27 1.27)) (justify left))
@@
     (pin "1")
   )
+  (symbol (lib_id "power:GND") (at 38.1 136.525 0) (unit 1)
+    (in_bom yes) (on_board yes)
+    (property "Reference" "#PWR0101" (id 0) (at 38.1 142.875 0)
+      (effects (font (size 1.27 1.27)) hide)
+    )
+    (property "Value" "GND" (id 1) (at 38.1 144.145 90)
+      (effects (font (size 1.27 1.27)) (justify left))
+    )
+    (property "Footprint" "" (id 2) (at 38.1 136.525 0)
+      (effects (font (size 1.27 1.27)) hide)
+    )
+    (property "Datasheet" "" (id 3) (at 38.1 136.525 0)
+      (effects (font (size 1.27 1.27)) hide)
+    )
+    (pin "1")
+  )
   (symbol (lib_id "Device:R_Small") (at 40.64 66.04 90) (mirror x) (unit 1)
     (in_bom yes) (on_board yes)
@@
     (pin "1")
     (pin "2")
-  )
-  (symbol (lib_id "Mechanical:MountingHole") (at 36.83 140.97 0) (unit 1)
-    (in_bom yes) (on_board yes) (fields_autoplaced)
-    (property "Reference" "H1" (id 0) (at 39.37 139.6999 0)
-      (effects (font (size 1.27 1.27)) (justify left))
-    )
-    (property "Value" "MountingHole" (id 1) (at 39.37 142.2399 0)
-      (effects (font (size 1.27 1.27)) (justify left))
-    )
-    (property "Footprint" "MountingHole:MountingHole_2.2mm_M2" (id 2) (at 36.83 140.97 0)
-      (effects (font (size 1.27 1.27)) hide)
-    )
-    (property "Datasheet" "~" (id 3) (at 36.83 140.97 0)
-      (effects (font (size 1.27 1.27)) hide)
-    )
   )
   (symbol (lib_id "power:GND") (at 120.65 99.06 90) (unit 1)
@@
     (pin "SH")
   )
+  (symbol (lib_id "Device:C_Small") (at 31.75 133.985 0) (mirror x) (unit 1)
+    (in_bom yes) (on_board yes) (fields_autoplaced)
+    (property "Reference" "C1" (id 0) (at 29.21 132.7085 0)
+      (effects (font (size 1.27 1.27)) (justify right))
+    )
+    (property "Value" "0.1u" (id 1) (at 29.21 135.2485 0)
+      (effects (font (size 1.27 1.27)) (justify right))
+    )
+    (property "Footprint" "00_KeyParts:C_1608_HandSolder" (id 2) (at 31.75 133.985 0)
+      (effects (font (size 1.27 1.27)) hide)
+    )
+    (property "Datasheet" "~" (id 3) (at 31.75 133.985 0)
+      (effects (font (size 1.27 1.27)) hide)
+    )
+    (pin "1")
+    (pin "2")
+  )
   (symbol (lib_id "Connector:RJ45_LED_Shielded_x2") (at 99.06 73.66 0) (mirror y) (unit 2)
     (in_bom yes) (on_board yes) (fields_autoplaced)
@@
     (pin "SH")
   )
+  (symbol (lib_id "Device:C_Small") (at 38.1 133.985 0) (unit 1)
+    (in_bom yes) (on_board yes) (fields_autoplaced)
+    (property "Reference" "C2" (id 0) (at 40.64 132.7212 0)
+      (effects (font (size 1.27 1.27)) (justify left))
+    )
+    (property "Value" "0.1u" (id 1) (at 40.64 135.2612 0)
+      (effects (font (size 1.27 1.27)) (justify left))
+    )
+    (property "Footprint" "00_KeyParts:C_1608_HandSolder" (id 2) (at 38.1 133.985 0)
+      (effects (font (size 1.27 1.27)) hide)
+    )
+    (property "Datasheet" "~" (id 3) (at 38.1 133.985 0)
+      (effects (font (size 1.27 1.27)) hide)
+    )
+    (pin "1")
+    (pin "2")
+  )
   (symbol (lib_id "power:GND") (at 99.06 86.36 0) (unit 1)
     (in_bom yes) (on_board yes)
@@
   )
   (symbol_instances
+    (path "/6e66920b-fd59-4940-8d81-ce066df9c8d7"
+      (reference "#PWR0101") (unit 1) (value "GND") (footprint "")
+    )
+    (path "/0cd33fa7-e147-4c4b-8417-ff91675a776f"
+      (reference "#PWR0102") (unit 1) (value "GND") (footprint "")
+    )
     (path "/5883adee-93fd-4737-8f82-f6684dad7ff7"
       (reference "#PWR0105") (unit 1) (value "GND") (footprint "")
@@
       (reference "#PWR0112") (unit 1) (value "GND") (footprint "")
     )
-    (path "/9dbd817f-0427-4793-ad42-e0834f0f29ce"
-      (reference "H1") (unit 1) (value "MountingHole") (footprint "MountingHole:MountingHole_2.2mm_M2")
+    (path "/b7567b6e-3de8-4b82-b23f-74dfaff46e72"
+      (reference "C1") (unit 1) (value "0.1u") (footprint "00_KeyParts:C_1608_HandSolder")
+    )
+    (path "/d694c1c5-91e5-4116-8a8e-47b086564ee3"
+      (reference "C2") (unit 1) (value "0.1u") (footprint "00_KeyParts:C_1608_HandSolder")
     )
     (path "/a74eea9b-8fa2-403b-a9b9-8d0507d5733d"

Commit message: i2c regs wip
Connections:
- net 5VD: now also C1.1; no longer C1.2
- net GND: now also C1.2; no longer C1.1
Changed lines of the file:
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@@
   )
   (symbol (lib_id "Seeeduino XIAO:SeeeduinoXIAO") (at 76.2 109.22 0) (unit 1)
-    (in_bom yes) (on_board yes) (fields_autoplaced)
+    (in_bom yes) (on_board no) (fields_autoplaced)
     (property "Reference" "U1" (id 0) (at 80.7594 130.81 0)
       (effects (font (size 1.27 1.27)) (justify left))
@@
     (pin "SH")
   )
-  (symbol (lib_id "Device:C_Small") (at 31.75 133.985 0) (mirror x) (unit 1)
-    (in_bom yes) (on_board yes) (fields_autoplaced)
-    (property "Reference" "C1" (id 0) (at 29.21 132.7085 0)
-      (effects (font (size 1.27 1.27)) (justify right))
-    )
-    (property "Value" "0.1u" (id 1) (at 29.21 135.2485 0)
-      (effects (font (size 1.27 1.27)) (justify right))
+  (symbol (lib_id "Device:C_Small") (at 31.75 133.985 0) (unit 1)
+    (in_bom yes) (on_board yes) (fields_autoplaced)
+    (property "Reference" "C1" (id 0) (at 34.29 132.7212 0)
+      (effects (font (size 1.27 1.27)) (justify left))
+    )
+    (property "Value" "0.1u" (id 1) (at 34.29 135.2612 0)
+      (effects (font (size 1.27 1.27)) (justify left))
     )
     (property "Footprint" "00_KeyParts:C_1608_HandSolder" (id 2) (at 31.75 133.985 0)
